File: VCAT/Kevin/kevin.kicad_pcb (KiCad board)
At the start: 4 copper layers, 0 parts

Commit message: second meeting meow
Parts:
- added C1: 4.7u, Capacitor_SMD:C_0603_1608Metric, F.Cu at (141.8, 69.6)
- added C10: 4.7u, Capacitor_SMD:C_0603_1608Metric, F.Cu at (145.0, 68.2)
- added C11: 100n, Capacitor_SMD:C_0402_1005Metric, F.Cu at (144.5, 69.5)
- added C12: 100n, Capacitor_SMD:C_0402_1005Metric, F.Cu at (152.0, 72.8)
- added C13: 100n, Capacitor_SMD:C_0402_1005Metric, F.Cu at (137.1, 87.6)
- added C14: 4.7u, Capacitor_SMD:C_0603_1608Metric, F.Cu at (148.0, 70.2)
- added C15: 10p, Capacitor_SMD:C_0402_1005Metric, F.Cu at (147.3, 81.4)
- added C16: 10p, Capacitor_SMD:C_0402_1005Metric, F.Cu at (143.3, 81.3)
- added C17: .8p, Capacitor_SMD:C_0402_1005Metric, F.Cu at (153.6, 74.4)
- added C18: .3p, Capacitor_SMD:C_0402_1005Metric, F.Cu at (155.6, 74.4)
- added C19: 100n, Capacitor_SMD:C_0402_1005Metric, F.Cu at (142.2, 85.2)
- added C2: 4.7u, Capacitor_SMD:C_0603_1608Metric, F.Cu at (136.0, 66.8)
- added C3: 4.7u, Capacitor_SMD:C_0603_1608Metric, F.Cu at (141.7, 81.0)
- added C4: 100n, Capacitor_SMD:C_0402_1005Metric, F.Cu at (140.3, 75.0)
- added C5: 100n, Capacitor_SMD:C_0402_1005Metric, F.Cu at (148.6, 79.8)
- added C6: 100n, Capacitor_SMD:C_0402_1005Metric, F.Cu at (142.4, 78.4)
- added C7: 100n, Capacitor_SMD:C_0402_1005Metric, F.Cu at (144.5, 70.5)
- added C8: 100n, Capacitor_SMD:C_0402_1005Metric, F.Cu at (151.9, 75.1)
- added C9: 100n, Capacitor_SMD:C_0402_1005Metric, F.Cu at (143.7, 79.8)
- added D1: USBLC6-2SC6, Package_TO_SOT_SMD:SOT-23-6, F.Cu at (139.4, 72.8)
- added D2: LED, LED_SMD:LED_0402_1005Metric, F.Cu at (152.8, 77.8)
- added FLT1: DLF162500LT-5028A1, Starter Footprint:DLF162500LT-5028A1, B.Cu at (156.6, 74.4)
- added FM1: Fiducial, Fiducial:Fiducial_1mm_Mask2mm, F.Cu at (138.0, 64.2)
- added FM2: Fiducial, Fiducial:Fiducial_1mm_Mask2mm, F.Cu at (137.8, 90.6)
- added FM3: Fiducial, Fiducial:Fiducial_1mm_Mask2mm, F.Cu at (158.0, 78.0)
- added H1: MountingHole_Pad, MountingHole:MountingHole_2.2mm_M2_Pad, F.Cu at (158.0, 90.0)
- added H2: MountingHole_Pad, MountingHole:MountingHole_2.2mm_M2_Pad, F.Cu at (132.0, 65.0)
- added H3: MountingHole_Pad, MountingHole:MountingHole_2.2mm_M2_Pad, F.Cu at (132.0, 89.8)
- added H4: MountingHole_Pad, MountingHole:MountingHole_2.2mm_M2_Pad, F.Cu at (158.0, 65.0)
- added J1: USB_C_Receptacle_USB2.0_16P, Connector_USB:USB_C_Receptacle_GCT_USB4105-xx-A_16P_TopMnt_Horizontal, F.Cu at (132.5, 73.0)
- added J2: Conn_01x04, Connector_Molex:Molex_PicoBlade_53048-0410_1x04_P1.25mm_Horizontal, F.Cu at (157.7, 81.5)
- added J3: Conn_ARM_SWD_TagConnect_TC2030, Connector:Tag-Connect_TC2030-IDC-FP_2x03_P1.27mm_Vertical, F.Cu at (136.7, 82.8)
- added J4: Conn_Coaxial, Connector_Coaxial:U.FL_Hirose_U.FL-R-SMT-1_Vertical, F.Cu at (156.2, 70.7)
- added L1: 10n, Inductor_SMD:L_0402_1005Metric, F.Cu at (146.0, 70.0)
- added L2: 10u, Inductor_SMD:L_0805_2012Metric, F.Cu at (148.4, 68.6)
- added L3: 2.7n, Inductor_SMD:L_0402_1005Metric, F.Cu at (154.6, 74.4)
- added R1: 5.1k, Resistor_SMD:R_0402_1005Metric, F.Cu at (138.8, 77.0)
- added R2: 5.1k, Resistor_SMD:R_0402_1005Metric, F.Cu at (138.4, 75.0)
- added R3: 220R, Resistor_SMD:R_0402_1005Metric, F.Cu at (150.6, 80.8)
- added R4: 220R, Resistor_SMD:R_0402_1005Metric, F.Cu at (151.8, 80.8)
- added R5: 220R, Resistor_SMD:R_0402_1005Metric, F.Cu at (153.8, 77.8)
- added R6: 5.1k, Resistor_SMD:R_0402_1005Metric, F.Cu at (142.2, 86.2)
- added R7: 220R, Resistor_SMD:R_0402_1005Metric, F.Cu at (143.8, 85.6)
- added SW1: SW_Push, Button_Switch_THT:SW_NKK_GW12LJP, F.Cu at (145.9, 86.0)
- added U1: MIC5365-3.3YD5, Package_TO_SOT_SMD:SOT-23-5, F.Cu at (139.2, 68.2)
- added U3: STM32WB55CEU6, Package_DFN_QFN:QFN-48-1EP_7x7mm_P0.5mm_EP5.6x5.6mm, F.Cu at (147.2, 75.1)
- added X1: 32.768kHz, Crystal:Crystal_SMD_2012-2Pin_2.0x1.2mm, F.Cu at (145.3, 81.4)
- added X2: 32mHz, Crystal:Crystal_SMD_2016-4Pin_2.0x1.6mm, F.Cu at (152.3, 69.9)
Routing:
- net GND: track 0.00 -> 83.1 mm, vias 0 -> 11
- net +3.3V: track 0.00 -> 32.2 mm, vias 0 -> 8
- net /SWD_NRST: track 0.00 -> 23.2 mm, vias 0 -> 2
- net /SWD_DIO: track 0.00 -> 19.8 mm, vias 0 -> 2
- net +5V: track 0.00 -> 19.7 mm, vias 0 -> 2
- net /SWD_CLK: track 0.00 -> 13.1 mm, vias 0 -> 2
- net /USB_D-: track 0.00 -> 11.0 mm
- net /USB_D+: track 0.00 -> 10.5 mm
- net /BOOT0: track 0.00 -> 10.3 mm, vias 0 -> 2
- net /SWD_TRC: track 0.00 -> 9.96 mm
- net /UART_TXC: track 0.00 -> 8.28 mm
- net /USB_CC1: track 0.00 -> 8.06 mm, vias 0 -> 2
- net /UART_RXC: track 0.00 -> 6.51 mm
- net /LSE_OUT: track 0.00 -> 4.56 mm
- net /LSE_IN: track 0.00 -> 4.51 mm
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- added copper zone on In2.Cu, net +3.3V
- added copper zone on In1.Cu, net GND
Other:
- board outline added: 32.1 x 30.8 mm
