File: VCAT/Kevin/kevin.kicad_sch (KiCad schematic)
At the start: 41 parts, among them J1 USB_C_Receptacle_USB2.0_16P, J2 Conn_ARM_SWD_TagConnect_TC2030, J3 Conn_01x04, J4 Conn_Coaxial, SW1 SW_Push, U1 MIC5365-3.3YD5, U2 USBLC6-2SC6, U3 STM32WB55CEU6, X1 32.768kHz, X2 32mHz

Commit message: second meeting meow
Parts:
- added FM1, FM2, FM3: Fiducial, Fiducial:Fiducial_1mm_Mask2mm, symbol Mechanical:Fiducial
- added H1, H2, H3, H4: MountingHole_Pad, MountingHole:MountingHole_2.2mm_M2_Pad, symbol Mechanical:MountingHole_Pad
- J2: renamed from J3; footprint Package_TO_SOT_SMD:TSOT-23-5 -> Connector_Molex:Molex_PicoBlade_53048-0410_1x04_P1.25mm_Horizontal
- J3: renamed from J2; footprint Connector_Molex:Molex_PicoBlade_53048-0410_1x04_P1.25mm_Horizontal -> Connector:Tag-Connect_TC2030-IDC-FP_2x03_P1.27mm_Vertical
- J4: footprint Connector:Tag-Connect_TC2030-IDC-FP_2x03_P1.27mm_Vertical -> Connector_Coaxial:U.FL_Hirose_U.FL-R-SMT-1_Vertical
- U1: footprint Button_Switch_SMD:SW_SPST_CK_RS282G05A3 -> Package_TO_SOT_SMD:SOT-23-5
- X2: footprint Connector_Coaxial:U.FL_Hirose_U.FL-R-SMT-1_Vertical -> Crystal:Crystal_SMD_2016-4Pin_2.0x1.6mm
- renumbered U2 to D1, D1 to D2
Connections:
- net +3.3V: now also U3.8 (VDDA)
- net LSE_OUT: now reaches C15.1, U3.3 (PC15), X1.1
- net LSE_IN: now reaches C16.1, U3.2 (PC14), X1.2
- net SMPS_LX: now reaches L1.1, U3.33 (VLXSMPS)
- net SMPS_LXL: now reaches L1.2, L2.1
- net SMPSFB renamed SMPS_FB
- net SWCLK4 renamed SWD_CLK
- net SWDIO renamed SWD_DIO
- net SWO renamed SWD_TRC
- no-connect marks 22 -> 25
Other:
- note added: "Mounting Holes and Fiducial Markers"
