File: VCAT/Dev/Project/STM32 Bluetooth.kicad_sch (KiCad schematic)
At the start: 41 parts, among them J1 USB_C_Receptacle_USB2.0, J2 Conn_01x04, J3 TC2030, J4 Conn_Coaxial, SW1 SW_Push, U1 MIC5365-3.3YD5, U2 USBLC6-2SC6, U3 STM32WB55CEU, X1 32kHz768, X2 32MHz

Commit message: final
Parts:
- added FM1, FM2, FM3: Fiducial, Fiducial:Fiducial_1mm_Mask2mm, symbol Mechanical:Fiducial
- added H1, H2, H3, H4: MountingHole_Pad, MountingHole:MountingHole_2.2mm_M2_Pad, symbol Mechanical:MountingHole_Pad
Connections:
- net GND: now also J4.2 (Ext), H1.1, H2.1, H3.1, H4.1
- net RF_ANT: now also J4.1 (In)
- net USB_D+: now also J1.A6 (D+), J1.B6 (D+), U2.3 (I/O2)
- net USB_D-: now also J1.A7 (D-), J1.B7 (D-), U2.1 (I/O1)
Other:
- moved on the sheet: J4
