File: VCAT/Dev/Project/STM32 Bluetooth.kicad_pcb (KiCad board)
At the start: 4 copper layers, 56 x 47.5 mm, 41 parts, among them J1 USB_C_Receptacle_USB2.0, J2 Conn_01x04, J3 TC2030, J4 Conn_Coaxial, SW1 SW_Push, U1 MIC5365-3.3YD5, U2 USBLC6-2SC6, U3 STM32WB55CEU, X1 32kHz768, X2 32MHz

Commit message: final
Parts:
- added FM1: Fiducial, Fiducial:Fiducial_1mm_Mask2mm, F.Cu at (73.4, 69.0)
- added FM2: Fiducial, Fiducial:Fiducial_1mm_Mask2mm, F.Cu at (112.9, 69.0)
- added FM3: Fiducial, Fiducial:Fiducial_1mm_Mask2mm, F.Cu at (65.4, 95.5)
- added H1: MountingHole_Pad, MountingHole:MountingHole_2.2mm_M2_Pad, F.Cu at (69.4, 69.5)
- added H2: MountingHole_Pad, MountingHole:MountingHole_2.2mm_M2_Pad, F.Cu at (69.4, 95.0)
- added H3: MountingHole_Pad, MountingHole:MountingHole_2.2mm_M2_Pad, F.Cu at (116.9, 70.0)
- added H4: MountingHole_Pad, MountingHole:MountingHole_2.2mm_M2_Pad, F.Cu at (116.4, 94.0)
- moved R1 11.4 mm to (85.3, 84.0)
- moved R2 10.7 mm to (85.3, 72.2)
- moved J1 10.6 mm to (81.5, 78.0)
- moved U2 9.96 mm to (88.8, 78.0)
- moved C4 9.19 mm to (95.6, 70.4)
- moved C2 5.06 mm to (84.8, 88.0), turned to -90 degrees
- moved C1 4.42 mm to (78.4, 87.7), turned to -90 degrees
- moved J3 3.99 mm to (90.6, 84.4)
- moved R4 3.19 mm to (103.0, 85.8), turned to 90 degrees
- moved C6 2.67 mm to (99.0, 75.0), turned to 90 degrees
- moved R6 2.58 mm to (99.2, 91.3), turned to -90 degrees
- moved R3 2.41 mm to (108.8, 81.8), turned to -90 degrees
- moved C3 2.36 mm to (107.3, 84.6)
- moved C5 2.22 mm to (105.9, 84.9)
- moved C13 2.04 mm to (102.3, 88.3), turned to -90 degrees
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Connections:
- J1 pad A6: Net-(J1-D+-PadA6) -> /USB_D+
- J1 pad A7: Net-(J1-D--PadA7) -> /USB_D-
- J1 pad B6: Net-(J1-D+-PadA6) -> /USB_D+
- J1 pad B7: Net-(J1-D--PadA7) -> /USB_D-
- U2 pad 1: Net-(J1-D--PadA7) -> /USB_D-
- U2 pad 3: Net-(J1-D+-PadA6) -> /USB_D+
Routing:
- net GND: track 0.00 -> 86.9 mm, vias 0 -> 36
- net +5V: track 0.00 -> 67.2 mm, vias 0 -> 4
- net /SWD_NRST: track 0.00 -> 28.3 mm
- net +3V3: track 0.00 -> 27.3 mm, vias 0 -> 14
- net /USB_D-: track 0.00 -> 14.7 mm
- net /USB_D+: track 0.00 -> 14.7 mm
- net /BOOT0: track 0.00 -> 12.9 mm, vias 0 -> 2
- net /SWD_TRC: track 0.00 -> 10.7 mm
- net /SMPSFB: track 0.00 -> 10.3 mm
- net Net-(J1-CC1): track 0.00 -> 9.53 mm
- net /SWD_DIO: track 0.00 -> 8.97 mm
- net /SWD_CLK: track 0.00 -> 8.50 mm
- net Net-(J1-CC2): track 0.00 -> 8.16 mm
- net /UART_TXC: track 0.00 -> 5.60 mm
- net /UART_RXC: track 0.00 -> 5.60 mm
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- added copper zone on B.Cu, net (none)
- added copper zone on In2.Cu, net +3V3
Other:
- board size 56 x 47.5 mm -> 56.1 x 31 mm

Commit message: donedone
Routing:
- net +5V: track 67.2 -> 6.44 mm, vias 4 -> 5
- net GND: track 86.9 -> 76.7 mm, vias 36 -> 30
- net +3V3: track 27.3 -> 29.7 mm
- added copper zone on B.Cu, net +5V
- added copper zone on F.Cu, net GND
- removed copper zone on B.Cu, net (none)

Commit message: for review:
Routing:
- net +5V: track 6.44 -> 7.58 mm
- net GND: track 76.7 -> 76.9 mm, vias 30 -> 32
Changed lines of the file:
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@@
+	)
+	(segment
+		(start 115.485 78.075)
+		(end 115.485 78.085)
+		(width 0.25)
+		(layer "F.Cu")
+		(net "GND")
 	)
 	(segment
@@
 	)
 	(segment
+		(start 115.485 81.025)
+		(end 115.4 81.025)
+		(width 0.25)
+		(layer "F.Cu")
+		(net "GND")
+	)
+	(segment
 		(start 93.0147 87.7853)
 		(end 93.1 87.7)
@@
 	)
 	(segment
+		(start 115.485 78.085)
+		(end 115.55 78.15)
+		(width 0.25)
+		(layer "F.Cu")
+		(net "GND")
+	)
+	(segment
 		(start 97.05 75.75)
 		(end 97.2 75.75)
@@
 	)
 	(via
+		(at 115.4 81.025)
+		(size 0.8)
+		(drill 0.4)
+		(layers "F.Cu" "B.Cu")
+		(net "GND")
+	)
+	(via
 		(at 78.43125 89.775)
 		(size 0.7)
@@
 		(size 0.7)
 		(drill 0.3)
+		(layers "F.Cu" "B.Cu")
+		(net "GND")
+	)
+	(via
+		(at 115.55 78.15)
+		(size 0.8)
+		(drill 0.4)
 		(layers "F.Cu" "B.Cu")
 		(net "GND")
@@
 	)
 	(segment
+		(start 79.425 87.175)
+		(end 79.35 87.1)
+		(width 0.25)
+		(layer "F.Cu")
+		(net "+5V")
+	)
+	(segment
 		(start 78.39375 86.95)
 		(end 79.2 86.95)
@@
 		(start 79.2 86.95)
 		(end 79.35 87.1)
+		(width 0.25)
+		(layer "F.Cu")
+		(net "+5V")
+	)
+	(segment
+		(start 80.45625 87.175)
+		(end 79.425 87.175)
 		(width 0.25)
 		(layer "F.Cu")
@@
 	)
 	(zone
+		(net "GND")
+		(layer "F.Cu")
+		(hatch edge 0.5)
+		(priority 4)
+		(connect_pads
+			(clearance 0.3)
+		)
+		(min_thickness 0.15)
+		(fill yes
+			(thermal_gap 0.4)
+			(thermal_bridge_width 0.25)
+			(island_removal_mode 0)
+		)
+		(polygon
+			(pts
+				(xy 114.05 80.35) (xy 114.495 80.3) (xy 117.4 80.5) (xy 117.5 82.5) (xy 114.05 82.35) (xy 114.1 80.35)
+			)
+		)
+	)
+	(zone
