File: PSYS/Gavin/Gavin_Starter.kicad_sch (KiCad schematic)
At the start: 41 parts, among them J1 Conn_Coaxial, J2 Conn_ARM_SWD_TagConnect_TC2030, J3 USB_C_Receptacle_USB2.0_16P, J4 Conn_01x04, SW1 SW_Push, U1 STM32WB55CEUx, U2 USBLC6-2SC6, U3 MIC5365-3.3YD5, X1 32MHz, X2 32Khz768

Commit message: schematic2
Parts:
- C8: value C -> 4u7
- C9: value C -> 100n
- J4: value Conn_01x04 -> UART_Connector
Connections:
- net GND: now also R4.2, U2.2 (GND); no longer R4.1
- net LED_A: now also D1.2 (A), U1.16 (PA7)
- net CC2: now reaches J3.B5 (CC2), R3.2
- net CC1: now reaches J3.A5 (CC1)
- net CC1: now also R4.1; no longer R4.2
- net SWD_DID renamed SWCLK
- net SWD_NRST renamed NRST
- net SWD_TRC renamed SWDIO
- net SWDIO: no longer J2.6 (SWO), U1.43 (PB3)
- new net SWO: J2.6 (SWO), U1.43 (PB3)
Other:
- note added: "Boot"
- note added: "Low Pass Filter"
- note added: "Test LED"
- note added: "mcu oscillator"
- note added: "radiofrequency component"
- moved on the sheet: C1, C10, C11, C14, C15, C16, C17, C18, C19, C2, C3, C4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

Commit message: Schematic3
Parts:
- C1, C10, C14, C15, C17, C2, C3, C4, C5, C6, C9: footprint (none) -> Capacitor_SMD:C_0402_1005Metric
- C11, C7, C8: footprint (none) -> Capacitor_SMD:C_0603_1608Metric
- C12, C13: value C -> 10p; footprint (none) -> Capacitor_SMD:C_0402_1005Metric
- C16: value C -> 100n; footprint (none) -> Capacitor_SMD:C_0402_1005Metric
- C18, C19: value C -> 4u7; footprint (none) -> Capacitor_SMD:C_0603_1608Metric
- D1: footprint (none) -> LED_SMD:LED_0402_1005Metric
- J1: footprint (none) -> Connector_Coaxial:U.FL_Hirose_U.FL-R-SMT-1_Vertical
- J3: footprint (none) -> Connector_USB:USB_C_Receptacle_GCT_USB4105-xx-A_16P_TopMnt_Horizontal
- J4: footprint (none) -> Connector_Molex:Molex_PicoBlade_53048-0410_1x04_P1.25mm_Horizontal
- L1, L3: footprint (none) -> Inductor_SMD:L_0402_1005Metric
- L2: footprint (none) -> Inductor_SMD:L_0805_2012Metric
- R1, R2, R3, R4, R5, R6, R7: footprint (none) -> Resistor_SMD:R_0402_1005Metric
- SW1: footprint (none) -> Button_Switch_SMD:SW_Push_1P1T_NO_CK_KMR2
- X1: footprint (none) -> Crystal:Crystal_SMD_2016-4Pin_2.0x1.6mm
- X2: footprint (none) -> Crystal:Crystal_SMD_2012-2Pin_2.0x1.2mm
Connections:
- no-connect marks 20 -> 21
Other:
- note added: "Decoupling Capacitors"
- note added: "UART Connector"
- moved on the sheet: C10, C16, C18, C19, C8, C9, J2, R3, R4, U3
