File: PSYS/Gavin/Gavin_Starter.kicad_pcb (KiCad board)
At the start: 4 copper layers, 0 parts

Commit message: layout
Parts:
- added C1: 100n, Capacitor_SMD:C_0402_1005Metric, F.Cu at (136.2, 114.1)
- added C10: 100n, Capacitor_SMD:C_0402_1005Metric, F.Cu at (139.0, 118.0)
- added C11: 4u7, Capacitor_SMD:C_0603_1608Metric, F.Cu at (156.5, 116.5)
- added C12: 10p, Capacitor_SMD:C_0402_1005Metric, F.Cu at (139.0, 120.0)
- added C13: 10p, Capacitor_SMD:C_0402_1005Metric, F.Cu at (139.0, 121.9)
- added C14: 0p8, Capacitor_SMD:C_0402_1005Metric, F.Cu at (141.9, 114.1)
- added C15: 0p3, Capacitor_SMD:C_0402_1005Metric, F.Cu at (141.9, 116.0)
- added C16: 100n, Capacitor_SMD:C_0402_1005Metric, F.Cu at (141.9, 118.0)
- added C17: 100n, Capacitor_SMD:C_0402_1005Metric, F.Cu at (141.9, 120.0)
- added C18: 4u7, Capacitor_SMD:C_0603_1608Metric, F.Cu at (156.5, 119.0)
- added C19: 4u7, Capacitor_SMD:C_0603_1608Metric, F.Cu at (156.5, 121.5)
- added C2: 100n, Capacitor_SMD:C_0402_1005Metric, F.Cu at (136.2, 116.0)
- added C3: 100n, Capacitor_SMD:C_0402_1005Metric, F.Cu at (136.2, 118.0)
- added C4: 100n, Capacitor_SMD:C_0402_1005Metric, F.Cu at (136.2, 120.0)
- added C5: 100n, Capacitor_SMD:C_0402_1005Metric, F.Cu at (136.2, 121.9)
- added C6: 100n, Capacitor_SMD:C_0402_1005Metric, F.Cu at (139.0, 114.1)
- added C7: 4u7, Capacitor_SMD:C_0603_1608Metric, F.Cu at (156.5, 111.5)
- added C8: 4u7, Capacitor_SMD:C_0603_1608Metric, F.Cu at (156.5, 114.0)
- added C9: 100n, Capacitor_SMD:C_0402_1005Metric, F.Cu at (139.0, 116.0)
- added D1: LED, LED_SMD:LED_0402_1005Metric, F.Cu at (156.5, 102.1)
- added FLT1: ~, Gavinstarter_footprints:DLF162500LT-5028A1, F.Cu at (160.8, 115.0)
- added J1: Conn_Coaxial, Connector_Coaxial:U.FL_Hirose_U.FL-R-SMT-1_Vertical, F.Cu at (141.5, 109.0)
- added J2: Conn_ARM_SWD_TagConnect_TC2030, Connector:Tag-Connect_TC2030-IDC-FP_2x03_P1.27mm_Vertical, F.Cu at (141.8, 101.3)
- added J3: USB_C_Receptacle_USB2.0_16P, Connector_USB:USB_C_Receptacle_GCT_USB4105-xx-A_16P_TopMnt_Horizontal, F.Cu at (142.8, 91.8)
- added J4: UART_Connector, Connector_Molex:Molex_PicoBlade_53048-0410_1x04_P1.25mm_Horizontal, F.Cu at (148.6, 98.6)
- added L1: 10n, Inductor_SMD:L_0402_1005Metric, F.Cu at (146.6, 115.7)
- added L2: 10u, Inductor_SMD:L_0805_2012Metric, F.Cu at (161.1, 112.3)
- added L3: 2n7, Inductor_SMD:L_0402_1005Metric, F.Cu at (146.6, 117.7)
- added R1: 5k1, Resistor_SMD:R_0402_1005Metric, F.Cu at (147.5, 109.0)
- added R2: 100R, Resistor_SMD:R_0402_1005Metric, F.Cu at (149.5, 115.7)
- added R3: 5k1, Resistor_SMD:R_0402_1005Metric, F.Cu at (149.5, 117.7)
- added R4: 5k1, Resistor_SMD:R_0402_1005Metric, F.Cu at (150.4, 109.0)
- added R5: 100R, Resistor_SMD:R_0402_1005Metric, F.Cu at (152.4, 115.7)
- added R6: 100R, Resistor_SMD:R_0402_1005Metric, F.Cu at (152.4, 117.7)
- added R7: 220R, Resistor_SMD:R_0402_1005Metric, F.Cu at (153.3, 109.0)
- added SW1: SW_Push, Button_Switch_SMD:SW_Push_1P1T_NO_CK_KMR2, F.Cu at (158.2, 98.8)
- added U1: STM32WB55CEUx, Package_DFN_QFN:QFN-48-1EP_7x7mm_P0.5mm_EP5.6x5.6mm, F.Cu at (153.7, 91.2)
- added U2: USBLC6-2SC6, Package_TO_SOT_SMD:SOT-23-6, F.Cu at (160.9, 88.9)
- added U3: MIC5365-3.3YD5, Package_TO_SOT_SMD:TSOT-23-5, F.Cu at (160.9, 93.5)
- added X1: 32MHz, Crystal:Crystal_SMD_2016-4Pin_2.0x1.6mm, F.Cu at (160.8, 105.9)
- added X2: 32Khz768, Crystal:Crystal_SMD_2012-2Pin_2.0x1.2mm, F.Cu at (160.8, 109.3)

Commit message: organizedlayout
Parts:
- moved J1 58.6 mm to (200.0, 105.5)
- moved C10 56.9 mm to (182.0, 80.8), turned to -90 degrees
- moved J4 56.3 mm to (198.7, 124.3), turned to -90 degrees
- moved C9 53.3 mm to (179.0, 80.8), turned to -90 degrees
- moved R6 51.2 mm to (202.5, 128.0)
- moved R5 51.0 mm to (202.5, 125.0)
- moved C15 50.7 mm to (191.5, 105.5)
- moved C5 50.3 mm to (165.0, 80.8), turned to -90 degrees
- moved C4 49.9 mm to (167.0, 80.8), turned to -90 degrees
- moved C3 49.6 mm to (169.0, 80.8), turned to -90 degrees
- moved C1 49.6 mm to (172.9, 80.8), turned to -90 degrees
- moved C2 49.5 mm to (170.9, 80.8), turned to -90 degrees
- moved L1 48.6 mm to (188.5, 91.0)
- moved C11 45.5 mm to (194.9, 92.2), turned to -90 degrees
- moved C12 44.2 mm to (183.0, 124.0), turned to -90 degrees
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